File: Copter_Transmitter.brd (EAGLE design)
At the start: 100 x 80 mm, 36 parts

Commit message: Transmitter finished
Parts:
- removed JOY_LEFT, JOY_RIGHT: JOYSTIK_EDGE, My_flight:JOYSTIK_EDGE
- added CA4, CA5: 1uF, MyAmSys:C_SMD_TA_A
- added LDO3.1: MCP1700, MyCMOSsensor:MCP1700
- added R6, R7: 10k, MyPowerComponents:SMD_2.1X1.25
- added U$11, U$12: JOYSTICK_MINI, My_flight:JOYSTICK_MINI
- C2, C3: value 0.1uF -> 47pF
- moved R2 153.9 mm to (83.8, 30.3), turned to 90 degrees
- moved R1 152.2 mm to (83.8, 28.4), turned to 90 degrees
- moved L1 151.3 mm to (83.8, 24.6), turned to 90 degrees
- moved R4 134.5 mm to (46.5, 8.75), flipped to the bottom, turned to 90 degrees
- moved C1 126.6 mm to (86.6, 23.6)
- moved R3 122.6 mm to (49.3, 34.5), flipped to the bottom
- moved C3 122.6 mm to (80.9, 31.3), turned to 180 degrees
- moved C2 122.0 mm to (80.9, 27.4)
- moved R5 121.3 mm to (34.1, 18.1), flipped to the bottom, turned to 270 degrees
- moved CA3 116.6 mm to (81.0, 22.6)
- moved U$10 114.9 mm to (65.1, 40.7), turned to 180 degrees
- moved C12 114.2 mm to (36.1, 11.4), flipped to the bottom, turned to 90 degrees
- moved C9 112.3 mm to (46.8, 18.9), turned to 270 degrees
- moved C7 110.5 mm to (46.8, 15.0), turned to 90 degrees
- moved C8 109.2 mm to (46.8, 20.6), turned to 270 degrees
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Connections:
- net +3V3: now also CA4.PLUS, LDO3.1.(2)OUT, U$11.K21, U$11.K22, U$11.V1, U$11.V2, U$12.K21, U$12.K22, U$12.V1, U$12.V2; no longer JOY_LEFT.VK, JOY_LEFT.VX, JOY_LEFT.VY, JOY_RIGHT.VK, JOY_RIGHT.VX, JOY_RIGHT.VY
- net +5V: now also CA5.PLUS, LDO3.1.(3)IN
- net AD0: now also U$11.S2; no longer JOY_LEFT.SX
- net AD1: now also U$11.S1; no longer JOY_LEFT.SY
- net AD2: now also U$12.S2; no longer JOY_RIGHT.SX
- net AD3: now also U$12.S1; no longer JOY_RIGHT.SY
- net GND: now also CA4.MINUS, CA5.MINUS, LDO3.1.(1)GND, R6.X2, R7.X2, U$11.C1, U$11.C2, U$11.C3, U$11.C4, U$11.G1, U$11.G2, U$12.C1, U$12.C2, U$12.C3, U$12.C4, U$12.G1, U$12.G2; no longer JOY_LEFT.GK, JOY_LEFT.GX, JOY_LEFT.GY, JOY_RIGHT.GK, JOY_RIGHT.GX, JOY_RIGHT.GY
- net KL: now also R7.X1, U$11.K11, U$11.K12; no longer JOY_LEFT.SK
- net KR: now also R6.X1, U$12.K11, U$12.K12; no longer JOY_RIGHT.SK
Routing:
- net +3V3: track 0.00 -> 226.2 mm, vias 0 -> 5
- net +5V: track 0.00 -> 130.5 mm, vias 0 -> 3
- net SCK2: track 0.00 -> 80.7 mm, vias 0 -> 2
- net AD2: track 0.00 -> 80.6 mm, vias 0 -> 3
- net MOSI2: track 0.00 -> 79.9 mm, vias 0 -> 2
- net DC: track 0.00 -> 67.1 mm, vias 0 -> 2
- net KL: track 0.00 -> 66.6 mm, vias 0 -> 1
- net AD1: track 0.00 -> 62.9 mm, vias 0 -> 1
- net AD3: track 0.00 -> 61.6 mm, vias 0 -> 2
- net CSN2: track 0.00 -> 53.8 mm, vias 0 -> 1
- net AD0: track 0.00 -> 52.9 mm, vias 0 -> 1
- net RST: track 0.00 -> 52.0 mm, vias 0 -> 2
- net KR: track 0.00 -> 51.4 mm, vias 0 -> 1
- net DM: track 0.00 -> 39.2 mm, vias 0 -> 1
- net DP: track 0.00 -> 39.0 mm, vias 0 -> 1
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- added copper zone on layer 1, net GND
- added copper zone on layer 16, net GND
Other:
- board size 100 x 80 mm -> 96.7 x 44 mm
