File: Copter_Transmitter.sch (EAGLE design)
At the start: 36 parts

Commit message: Transmitter finished
Parts:
- removed JOY_LEFT, JOY_RIGHT: JOYSTIK_EDGE, My_flight:JOYSTIK_EDGE
- added CA4, CA5: 1uF, MyAmSys:C_SMD_TA_A
- added LDO3.1: MCP1700, MyCMOSsensor:MCP1700
- added R6, R7: 10k, MyPowerComponents:R_SMD_2.1X1.25
- added U$11, U$12: JOYSTICK_MINI, My_flight:JOYSTICK_MINI
- C2, C3: value 0.1uF -> 47pF
Connections:
- net +3V3: now also CA4.X2, LDO3.1.(2)OUT, U$11.K21, U$11.K22, U$11.V1, U$11.V2, U$12.K21, U$12.K22, U$12.V1, U$12.V2; no longer JOY_LEFT.VK, JOY_LEFT.VX, JOY_LEFT.VY, JOY_RIGHT.VK, JOY_RIGHT.VX, JOY_RIGHT.VY
- net +5V: now also CA5.X2, LDO3.1.(3)IN
- net AD0: now also U$11.S2; no longer JOY_LEFT.SX
- net AD1: now also U$11.S1; no longer JOY_LEFT.SY
- net AD2: now also U$12.S2; no longer JOY_RIGHT.SX
- net AD3: now also U$12.S1; no longer JOY_RIGHT.SY
- net GND: now also CA4.X1, CA5.X1, LDO3.1.(1)GND, R6.X2, R7.X2, U$11.C1, U$11.C2, U$11.C3, U$11.C4, U$11.G1, U$11.G2, U$12.C1, U$12.C2, U$12.C3, U$12.C4, U$12.G1, U$12.G2; no longer JOY_LEFT.GK, JOY_LEFT.GX, JOY_LEFT.GY, JOY_RIGHT.GK, JOY_RIGHT.GX, JOY_RIGHT.GY
- net KL: now also R7.X1, U$11.K11, U$11.K12; no longer JOY_LEFT.SK
- net KR: now also R6.X1, U$12.K11, U$12.K12; no longer JOY_RIGHT.SK
